Commit message: fixed mesh paths

File: urdf/iiwa14_macro.xacro (robot description, xacro)
@@ -21,5 +21,5 @@
                 <origin rpy="0 0 0" xyz="0 0 0" />
                 <geometry>
-                    <mesh filename="package://iiwa14_description/meshes/iiwa14/visual/link_0.dae" />
+                    <mesh filename="package://iiwa14_description/meshes/visual/link_0.dae" />
                 </geometry>
             </visual>
@@ -27,5 +27,5 @@
                 <origin rpy="0 0 0" xyz="0 0 0" />
                 <geometry>
-                    <mesh filename="package://iiwa14_description/meshes/iiwa14/collision/link_0.stl" />
+                    <mesh filename="package://iiwa14_description/meshes/collision/link_0.stl" />
                 </geometry>
             </collision>
@@ -58,5 +58,5 @@
                 <origin rpy="0 0 0" xyz="0.0 0.0 -0.1475" />
                 <geometry>
-                    <mesh filename="package://iiwa14_description/meshes/iiwa14/visual/link_1.dae" />
+                    <mesh filename="package://iiwa14_description/meshes/visual/link_1.dae" />
                 </geometry>
             </visual>
@@ -64,5 +64,5 @@
                 <origin rpy="0 0 0" xyz="0.0 0.0 -0.1475" />
                 <geometry>
-                    <mesh filename="package://iiwa14_description/meshes/iiwa14/collision/link_1.stl" />
+                    <mesh filename="package://iiwa14_description/meshes/collision/link_1.stl" />
                 </geometry>
             </collision>
@@ -95,5 +95,5 @@
                 <origin rpy="0 0 0" xyz="0.0 0.01 -0.36" />
                 <geometry>
-                    <mesh filename="package://iiwa14_description/meshes/iiwa14/visual/link_2.dae" />
+                    <mesh filename="package://iiwa14_description/meshes/visual/link_2.dae" />
                 </geometry>
             </visual>
@@ -101,5 +101,5 @@
                 <origin rpy="0 0 0" xyz="0.0 0.01 -0.36" />
                 <geometry>
-                    <mesh filename="package://iiwa14_description/meshes/iiwa14/collision/link_2.stl" />
+                    <mesh filename="package://iiwa14_description/meshes/collision/link_2.stl" />
                 </geometry>
             </collision>
@@ -132,5 +132,5 @@
                 <origin rpy="0 0 0" xyz="0.0 0.0 -0.588" />
                 <geometry>
-                    <mesh filename="package://iiwa14_description/meshes/iiwa14/visual/link_3.dae" />
+                    <mesh filename="package://iiwa14_description/meshes/visual/link_3.dae" />
                 </geometry>
             </visual>
@@ -138,5 +138,5 @@
                 <origin rpy="0 0 0" xyz="0.0 0.0 -0.588" />
                 <geometry>
-                    <mesh filename="package://iiwa14_description/meshes/iiwa14/collision/link_3.stl" />
+                    <mesh filename="package://iiwa14_description/meshes/collision/link_3.stl" />
                 </geometry>
             </collision>
@@ -169,5 +169,5 @@
                 <origin rpy="0 0 0" xyz="0.0 -0.0105 -0.78" />
                 <geometry>
-                    <mesh filename="package://iiwa14_description/meshes/iiwa14/visual/link_4.dae" />
+                    <mesh filename="package://iiwa14_description/meshes/visual/link_4.dae" />
                 </geometry>
             </visual>
@@ -175,5 +175,5 @@
                 <origin rpy="0 0 0" xyz="0.0 -0.0105 -0.78" />
                 <geometry>
-                    <mesh filename="package://iiwa14_description/meshes/iiwa14/collision/link_4.stl" />
+                    <mesh filename="package://iiwa14_description/meshes/collision/link_4.stl" />
                 </geometry>
             </collision>
@@ -206,5 +206,5 @@
                 <origin rpy="0 0 0" xyz="0.0 0.0 -0.9875" />
                 <geometry>
-                    <mesh filename="package://iiwa14_description/meshes/iiwa14/visual/link_5.dae" />
+                    <mesh filename="package://iiwa14_description/meshes/visual/link_5.dae" />
                 </geometry>
             </visual>
@@ -212,5 +212,5 @@
                 <origin rpy="0 0 0" xyz="0.0 0.0 -0.9875" />
                 <geometry>
-                    <mesh filename="package://iiwa14_description/meshes/iiwa14/collision/link_5.stl" />
+                    <mesh filename="package://iiwa14_description/meshes/collision/link_5.stl" />
                 </geometry>
             </collision>
@@ -243,5 +243,5 @@
                 <origin rpy="0 0 0" xyz="0.0 0.0707 -1.18" />
                 <geometry>
-                    <mesh filename="package://iiwa14_description/meshes/iiwa14/visual/link_6.dae" />
+                    <mesh filename="package://iiwa14_description/meshes/visual/link_6.dae" />
                 </geometry>
             </visual>
@@ -249,5 +249,5 @@
                 <origin rpy="0 0 0" xyz="0.0 0.0707 -1.18" />
                 <geometry>
-                    <mesh filename="package://iiwa14_description/meshes/iiwa14/collision/link_6.stl" />
+                    <mesh filename="package://iiwa14_description/meshes/collision/link_6.stl" />
                 </geometry>
             </collision>
@@ -279,5 +279,5 @@
                 <origin rpy="0 0 0" xyz="0.0 0.0 -1.271" />
                 <geometry>
-                    <mesh filename="package://iiwa14_description/meshes/iiwa14/visual/link_7.dae" />
+                    <mesh filename="package://iiwa14_description/meshes/visual/link_7.dae" />
                 </geometry>
             </visual>
@@ -285,5 +285,5 @@
                 <origin rpy="0 0 0" xyz="0.0 0.0 -1.271" />
                 <geometry>
-                    <mesh filename="package://iiwa14_description/meshes/iiwa14/collision/link_7.stl" />
+                    <mesh filename="package://iiwa14_description/meshes/collision/link_7.stl" />
                 </geometry>
             </collision>
